Commit message: 一键抓取成功，后续优化抓取角度问题

File: src/fairino3mt_v6_moveit2_config/config/fairino3mt_v6_robot.ros2_control.xacro (robot description, xacro)
@@ -1,10 +1,15 @@
 <?xml version="1.0"?>
 <robot xmlns:xacro="http://www.ros.org/wiki/xacro">
-    <xacro:macro name="fairino3mt_v6_robot_ros2_control" params="name initial_positions_file">
+    <xacro:macro name="fairino3mt_v6_robot_ros2_control" params="name initial_positions_file hardware_plugin">
         <xacro:property name="initial_positions" value="${load_yaml(initial_positions_file)['initial_positions']}"/>
         <ros2_control name="${name}" type="system">
             <hardware>
-                <!-- By default, set up controllers for simulation. This won't work on real hardware -->
-                <plugin>fairino_hardware/FairinoHardwareInterface</plugin>
+                <plugin>${hardware_plugin}</plugin>
+                <xacro:if value="${hardware_plugin == 'fairino_hardware/FairinoHardwareInterface'}">
+                  <param name="controller_ip">192.168.58.2</param>
+                  <!-- FAIRINO V3.9.2's official ROS 2 plugin sends ServoJ with cmdT=8 ms. -->
+                  <param name="servo_command_period_sec">0.008</param>
+                  <param name="control_period_tolerance_sec">0.002</param>
+                </xacro:if>
             </hardware>
             <joint name="joint1">
@@ -44,4 +49,46 @@
                 </state_interface>
             </joint>
+            <!-- Read-only FAIRINO controller state exported by the existing
+                 hardware connection. P6 consumes this through
+                 /dynamic_joint_states; it does not create a second SDK client. -->
+            <xacro:if value="${hardware_plugin == 'fairino_hardware/FairinoHardwareInterface'}">
+              <gpio name="fairino_status">
+                <state_interface name="program_state"/>
+                <state_interface name="robot_state"/>
+                <state_interface name="main_error_code"/>
+                <state_interface name="sub_error_code"/>
+                <state_interface name="robot_mode"/>
+                <state_interface name="tool_id"/>
+                <state_interface name="work_object_id"/>
+                <state_interface name="emergency_stop"/>
+                <state_interface name="motion_done"/>
+                <state_interface name="collision_state"/>
+                <state_interface name="safety_stop_0"/>
+                <state_interface name="safety_stop_1"/>
+                <state_interface name="enabled"/>
+                <state_interface name="payload_kg"/>
+                <state_interface name="payload_cog_x_mm"/>
+                <state_interface name="payload_cog_y_mm"/>
+                <state_interface name="payload_cog_z_mm"/>
+                <state_interface name="tool_x_mm"/>
+                <state_interface name="tool_y_mm"/>
+                <state_interface name="tool_z_mm"/>
+                <state_interface name="tool_rx_deg"/>
+                <state_interface name="tool_ry_deg"/>
+                <state_interface name="tool_rz_deg"/>
+                <state_interface name="wobj_x_mm"/>
+                <state_interface name="wobj_y_mm"/>
+                <state_interface name="wobj_z_mm"/>
+                <state_interface name="wobj_rx_deg"/>
+                <state_interface name="wobj_ry_deg"/>
+                <state_interface name="wobj_rz_deg"/>
+                <state_interface name="flange_x_mm"/>
+                <state_interface name="flange_y_mm"/>
+                <state_interface name="flange_z_mm"/>
+                <state_interface name="flange_rx_deg"/>
+                <state_interface name="flange_ry_deg"/>
+                <state_interface name="flange_rz_deg"/>
+              </gpio>
+            </xacro:if>
         </ros2_control>
     </xacro:macro>

File: src/fairino3mt_v6_moveit2_config/config/fairino3mt_v6_robot.urdf.xacro (robot description, xacro)
@@ -2,4 +2,5 @@
 <robot xmlns:xacro="http://www.ros.org/wiki/xacro" name="fairino3mt_v6_robot">
     <xacro:arg name="initial_positions_file" default="initial_positions.yaml" />
+    <xacro:arg name="hardware_plugin" default="fairino_hardware/FairinoHardwareInterface" />
     <!-- FR3-C controller FK matches the standard FAIRINO FR3 chain, not the
          fairino3_mt_v6 chain.  fairino3c_v6 is a joint-name-compatible copy
@@ -18,22 +19,50 @@
     <xacro:arg name="gripper_mount_rpy" default="0 0 0"/>
     <xacro:arg name="gripper_spacer" default="0.003"/>
-    <!-- Final practical TCP v2, 2026-09-10.  X/Y come from the 12-pose pivot
-         solve; flange-to-tip Z is the user's direct 178 mm measurement.  The
-         body-relative Z subtracts the retained 3 mm collision placeholder. -->
-    <xacro:arg name="gripper_tcp_from_body_xyz" default="-0.000847397 0.003027928 0.175"/>
+    <!-- Active TCP v3 table-contact test, 2026-09-11. All XYZ components come
+         from the 12-pose pivot solution. The 184.614459 mm flange-relative Z
+         matches the observed ~6 mm RViz shortfall of the prior 178 mm TCP.
+         Load the machine-readable calibration as the single source of truth;
+         body-relative Z subtracts the retained 3 mm collision spacer. -->
+    <xacro:property name="gripper_tcp_config"
+      value="${xacro.load_yaml('$(find fairino3mt_v6_moveit2_config)/config/ydi_j22_tcp.yaml')['ydi_j22_tcp']}"/>
+    <xacro:property name="gripper_tcp_flange_xyz" value="${gripper_tcp_config['xyz_m']}"/>
+    <xacro:property name="gripper_spacer_m" value="${float('$(arg gripper_spacer)')}"/>
+    <xacro:property name="gripper_tcp_from_body_xyz"
+      value="${'%s %s %s' % (gripper_tcp_flange_xyz[0], gripper_tcp_flange_xyz[1], gripper_tcp_flange_xyz[2] - gripper_spacer_m)}"/>
     <xacro:arg name="gripper_tcp_rpy" default="0 0 0"/>
-    <xacro:arg name="gripper_envelope_x" default="0.180"/>
-    <xacro:arg name="gripper_envelope_y" default="0.100"/>
-    <xacro:arg name="gripper_envelope_z" default="0.200"/>
+    <!-- First-grasp simplified collision geometry. Housing cross-section is
+         based on the 56 x 80.59 mm drawing. Finger tips end at the calibrated
+         TCP instead of extending 25 mm beyond it as the old solid box did. -->
+    <xacro:arg name="gripper_body_x" default="0.056"/>
+    <xacro:arg name="gripper_body_y" default="0.08059"/>
+    <xacro:arg name="gripper_body_z" default="0.085"/>
+    <xacro:arg name="gripper_finger_x" default="0.012"/>
+    <xacro:arg name="gripper_finger_y" default="0.013"/>
+    <xacro:property name="gripper_finger_proximal_body_z" value="${0.080}"/>
+    <xacro:property name="gripper_finger_z"
+      value="${gripper_tcp_flange_xyz[2] - gripper_spacer_m - gripper_finger_proximal_body_z}"/>
+    <xacro:arg name="gripper_finger_center_x" default="0.0205"/>
+    <xacro:arg name="gripper_finger_center_y" default="0.021"/>
+    <xacro:property name="gripper_finger_center_z"
+      value="${gripper_finger_proximal_body_z + gripper_finger_z / 2.0}"/>
+    <!-- (166 mm max span - 53 mm nominal grasp span) / (2 * 130 mm command). -->
+    <xacro:arg name="gripper_finger_open_multiplier" default="0.434615"/>
     <xacro:include filename="$(find fairino_description)/urdf/ydi_j22_placeholder.xacro"/>
       <xacro:ydi_j22_placeholder parent="flange_link"
         mount_xyz="$(arg gripper_mount_xyz)" mount_rpy="$(arg gripper_mount_rpy)"
-        spacer="$(arg gripper_spacer)" tcp_xyz="$(arg gripper_tcp_from_body_xyz)"
-        tcp_rpy="$(arg gripper_tcp_rpy)" envelope_x="$(arg gripper_envelope_x)"
-        envelope_y="$(arg gripper_envelope_y)" envelope_z="$(arg gripper_envelope_z)"/>
+        spacer="$(arg gripper_spacer)" tcp_xyz="${gripper_tcp_from_body_xyz}"
+        tcp_rpy="$(arg gripper_tcp_rpy)"
+        body_x="$(arg gripper_body_x)" body_y="$(arg gripper_body_y)"
+        body_z="$(arg gripper_body_z)" finger_x="$(arg gripper_finger_x)"
+        finger_y="$(arg gripper_finger_y)" finger_z="${gripper_finger_z}"
+        finger_center_x="$(arg gripper_finger_center_x)"
+        finger_center_y="$(arg gripper_finger_center_y)"
+        finger_center_z="${gripper_finger_center_z}"
+        finger_open_multiplier="$(arg gripper_finger_open_multiplier)"/>
     <!-- Camera housing: 100 x 35 x 20 mm measured by user.
          Centre offset estimated from photos, NOT a hand-eye calibration. -->
-    <!-- Nominal flange radius 40 mm + half camera height 17.5 mm. -->
-    <xacro:arg name="camera_mount_xyz" default="0 0.0575 0.015"/>
+    <!-- Nominal flange radius 40 mm + half camera height 17.5 mm. The camera
+         is physically on flange -Y; +Y was the earlier photo-based guess. -->
+    <xacro:arg name="camera_mount_xyz" default="0 -0.0575 0.015"/>
     <xacro:arg name="camera_mount_rpy" default="0 0 0"/>
     <xacro:arg name="camera_size_x" default="0.100"/>
@@ -48,4 +77,6 @@
     <!-- Import control_xacro -->
     <xacro:include filename="fairino3mt_v6_robot.ros2_control.xacro" />
-    <xacro:fairino3mt_v6_robot_ros2_control name="FakeSystem" initial_positions_file="$(arg initial_positions_file)"/>
+    <xacro:fairino3mt_v6_robot_ros2_control name="FR3CHardware"
+      initial_positions_file="$(arg initial_positions_file)"
+      hardware_plugin="$(arg hardware_plugin)"/>
 </robot>

File: src/fairino_description/urdf/ydi_j22_placeholder.xacro (robot description, xacro)
@@ -1,8 +1,17 @@
 <?xml version="1.0"?>
 <robot xmlns:xacro="http://www.ros.org/wiki/xacro">
-  <!-- Fixed planning placeholder, NOT a calibrated model of finger deformation.
-       Dimensions are metres.  The caller supplies the calibrated TCP separately
-       from the approximate visual/collision geometry. -->
-  <xacro:macro name="ydi_j22_placeholder" params="parent mount_xyz mount_rpy spacer tcp_xyz tcp_rpy envelope_x envelope_y envelope_z">
+  <!-- Simplified YDI-J22 model for the first 30 mm cube grasp.
+       The calibrated TCP is independent of this approximate geometry. The
+       body uses the manufacturer's 56 x 80.59 mm cross-section. Four named
+       finger links replace the former solid envelope so the grasp opening is
+       real collision-free space and contact permission can be limited to the
+       fingers. The finger motion is a planning approximation: all four
+       fingers move symmetrically in X from a nominal 29 mm closed opening to
+       the drawing's 166 mm maximum span. -->
+  <xacro:macro name="ydi_j22_placeholder"
+               params="parent mount_xyz mount_rpy spacer tcp_xyz tcp_rpy
+                       body_x body_y body_z finger_x finger_y finger_z
+                       finger_center_x finger_center_y finger_center_z
+                       finger_open_multiplier">
     <link name="gripper_mount_link"/>
     <joint name="gripper_mount_joint" type="fixed">
@@ -11,40 +20,90 @@
     </joint>
     <link name="gripper_spacer_link">
-      <visual><origin xyz="0 0 ${spacer/2}"/><geometry><box size="0.056 0.056 ${spacer}"/></geometry><material name="spacer_gray"><color rgba="0.55 0.55 0.55 1"/></material></visual>
-      <collision><origin xyz="0 0 ${spacer/2}"/><geometry><box size="0.056 0.056 ${spacer}"/></geometry></collision>
+      <visual>
+        <origin xyz="0 0 ${spacer/2}"/>
+        <geometry><box size="0.056 0.056 ${spacer}"/></geometry>
+        <material name="spacer_gray"><color rgba="0.55 0.55 0.55 1"/></material>
+      </visual>
+      <collision>
+        <origin xyz="0 0 ${spacer/2}"/>
+        <geometry><box size="0.056 0.056 ${spacer}"/></geometry>
+      </collision>
     </link>
-    <joint name="gripper_spacer_joint" type="fixed"><parent link="gripper_mount_link"/><child link="gripper_spacer_link"/></joint>
+    <joint name="gripper_spacer_joint" type="fixed">
+      <parent link="gripper_mount_link"/><child link="gripper_spacer_link"/>
+    </joint>
+    <!-- Fixed housing/servo region only; it no longer fills the finger opening. -->
     <link name="gripper_link">
-      <visual><origin xyz="0 0 0.0425"/><geometry><box size="0.056 0.081 0.085"/></geometry><material name="gripper_gray"><color rgba="0.35 0.38 0.42 1"/></material></visual>
-      <visual><origin xyz="0.049207 0.021 0.116843" rpy="0 0.65 0"/><geometry><box size="0.012 0.013 0.080"/></geometry><material name="finger_orange"><color rgba="0.85 0.45 0.12 1"/></material></visual>
-      <visual><origin xyz="0.049207 -0.021 0.116843" rpy="0 0.65 0"/><geometry><box size="0.012 0.013 0.080"/></geometry><material name="finger_orange"><color rgba="0.85 0.45 0.12 1"/></material></visual>
-      <visual><origin xyz="-0.049207 0.021 0.116843" rpy="0 -0.65 0"/><geometry><box size="0.012 0.013 0.080"/></geometry><material name="finger_orange"><color rgba="0.85 0.45 0.12 1"/></material></visual>
-      <visual><origin xyz="-0.049207 -0.021 0.116843" rpy="0 -0.65 0"/><geometry><box size="0.012 0.013 0.080"/></geometry><material name="finger_orange"><color rgba="0.85 0.45 0.12 1"/></material></visual>
-      <!-- A single conservative placeholder intentionally fills the grasp opening.
-           It is for clearance planning, not contact-aware pick/place. -->
-      <collision><origin xyz="0 0 ${envelope_z/2}"/><geometry><box size="${envelope_x} ${envelope_y} ${envelope_z}"/></geometry></collision>
+      <visual>
+        <origin xyz="0 0 ${body_z/2}"/>
+        <geometry><box size="${body_x} ${body_y} ${body_z}"/></geometry>
+        <material name="gripper_gray"><color rgba="0.35 0.38 0.42 1"/></material>
+      </visual>
+      <collision>
+        <origin xyz="0 0 ${body_z/2}"/>
+        <geometry><box size="${body_x} ${body_y} ${body_z}"/></geometry>
+      </collision>
     </link>
-    <joint name="gripper_joint" type="fixed"><parent link="gripper_spacer_link"/><child link="gripper_link"/><origin xyz="0 0 ${spacer}"/></joint>
-    <!-- Calibrated grasp TCP at the common flexible-finger closing tip.
-         tcp_xyz is expressed from gripper_link.  The caller compensates the
-         placeholder spacer so the complete flange transform remains the
-         fixed-point measurement. -->
-    <link name="grasp_frame"/>
-    <joint name="gripper_to_grasp_frame" type="fixed">
-      <parent link="gripper_link"/>
-      <child link="grasp_frame"/>
-      <origin xyz="${tcp_xyz}" rpy="${tcp_rpy}"/>
+    <joint name="gripper_joint" type="fixed">
+      <parent link="gripper_spacer_link"/><child link="gripper_link"/>
+      <origin xyz="0 0 ${spacer}"/>
     </joint>
-    <!-- Command/state-only joint for MoveIt GripperCommand integration.  It
-         carries no geometry: the deformable four-finger collision envelope
-         remains conservative until measured open/closed meshes are supplied. -->
+    <!-- Single command variable retained for the real GripperCommand driver. -->
     <link name="gripper_command_link"/>
     <joint name="gripper_command_joint" type="prismatic">
-      <parent link="gripper_link"/>
-      <child link="gripper_command_link"/>
+      <parent link="gripper_link"/><child link="gripper_command_link"/>
       <origin xyz="0 0 0" rpy="0 0 0"/>
       <axis xyz="1 0 0"/>
       <limit lower="0.0" upper="0.130" effort="1.0" velocity="0.130"/>
     </joint>
+    <!-- Four independently named contact links. Mimic joints make the two X
+         sides move apart symmetrically without adding control variables. -->
+    <link name="gripper_finger_px_py_link">
+      <visual><geometry><box size="${finger_x} ${finger_y} ${finger_z}"/></geometry><material name="finger_orange"><color rgba="0.85 0.45 0.12 1"/></material></visual>
+      <collision><geometry><box size="${finger_x} ${finger_y} ${finger_z}"/></geometry></collision>
+    </link>
+    <joint name="gripper_finger_px_py_joint" type="prismatic">
+      <parent link="gripper_link"/><child link="gripper_finger_px_py_link"/>
+      <origin xyz="${finger_center_x} ${finger_center_y} ${finger_center_z}"/>
+      <axis xyz="1 0 0"/><limit lower="0" upper="0.057" effort="1" velocity="0.057"/>
+      <mimic joint="gripper_command_joint" multiplier="${finger_open_multiplier}"/>
+    </joint>
+    <link name="gripper_finger_px_ny_link">
+      <visual><geometry><box size="${finger_x} ${finger_y} ${finger_z}"/></geometry><material name="finger_orange"/></visual>
+      <collision><geometry><box size="${finger_x} ${finger_y} ${finger_z}"/></geometry></collision>
+    </link>
+    <joint name="gripper_finger_px_ny_joint" type="prismatic">
+      <parent link="gripper_link"/><child link="gripper_finger_px_ny_link"/>
+      <origin xyz="${finger_center_x} ${-finger_center_y} ${finger_center_z}"/>
+      <axis xyz="1 0 0"/><limit lower="0" upper="0.057" effort="1" velocity="0.057"/>
+      <mimic joint="gripper_command_joint" multiplier="${finger_open_multiplier}"/>
+    </joint>
+    <link name="gripper_finger_nx_py_link">
+      <visual><geometry><box size="${finger_x} ${finger_y} ${finger_z}"/></geometry><material name="finger_orange"/></visual>
+      <collision><geometry><box size="${finger_x} ${finger_y} ${finger_z}"/></geometry></collision>
+    </link>
+    <joint name="gripper_finger_nx_py_joint" type="prismatic">
+      <parent link="gripper_link"/><child link="gripper_finger_nx_py_link"/>
+      <origin xyz="${-finger_center_x} ${finger_center_y} ${finger_center_z}"/>
+      <axis xyz="-1 0 0"/><limit lower="0" upper="0.057" effort="1" velocity="0.057"/>
+      <mimic joint="gripper_command_joint" multiplier="${finger_open_multiplier}"/>
+    </joint>
+    <link name="gripper_finger_nx_ny_link">
+      <visual><geometry><box size="${finger_x} ${finger_y} ${finger_z}"/></geometry><material name="finger_orange"/></visual>
+      <collision><geometry><box size="${finger_x} ${finger_y} ${finger_z}"/></geometry></collision>
+    </link>
+    <joint name="gripper_finger_nx_ny_joint" type="prismatic">
+      <parent link="gripper_link"/><child link="gripper_finger_nx_ny_link"/>
+      <origin xyz="${-finger_center_x} ${-finger_center_y} ${finger_center_z}"/>
+      <axis xyz="-1 0 0"/><limit lower="0" upper="0.057" effort="1" velocity="0.057"/>
+      <mimic joint="gripper_command_joint" multiplier="${finger_open_multiplier}"/>
+    </joint>
+    <!-- Calibrated common fingertip TCP. The parent model supplies the active
+         flange-relative value minus its retained 3 mm collision spacer. -->
+    <link name="grasp_frame"/>
+    <joint name="gripper_to_grasp_frame" type="fixed">
+      <parent link="gripper_link"/><child link="grasp_frame"/>
+      <origin xyz="${tcp_xyz}" rpy="${tcp_rpy}"/>
+    </joint>
   </xacro:macro>
 </robot>
