Commit message: 进行qwen开发

File: src/fairino3mt_v6_moveit2_config/config/fairino3mt_v6_robot.urdf.xacro (robot description, xacro)
@@ -37,4 +37,6 @@
     <xacro:arg name="gripper_body_y" default="0.08059"/>
     <xacro:arg name="gripper_body_z" default="0.085"/>
+    <!-- One-sided collision margin on the +Y face, away from the -Y camera. -->
+    <xacro:arg name="gripper_away_from_camera_collision_extension" default="0.005"/>
     <xacro:arg name="gripper_finger_x" default="0.012"/>
     <xacro:arg name="gripper_finger_y" default="0.013"/>
@@ -54,5 +56,7 @@
         tcp_rpy="$(arg gripper_tcp_rpy)"
         body_x="$(arg gripper_body_x)" body_y="$(arg gripper_body_y)"
-        body_z="$(arg gripper_body_z)" finger_x="$(arg gripper_finger_x)"
+        body_z="$(arg gripper_body_z)"
+        body_positive_y_collision_extension="$(arg gripper_away_from_camera_collision_extension)"
+        finger_x="$(arg gripper_finger_x)"
         finger_y="$(arg gripper_finger_y)" finger_z="${gripper_finger_z}"
         finger_center_x="$(arg gripper_finger_center_x)"
@@ -60,13 +64,15 @@
         finger_center_z="${gripper_finger_center_z}"
         finger_open_multiplier="$(arg gripper_finger_open_multiplier)"/>
-    <!-- Camera housing: 100 x 35 x 20 mm measured by user.
-         Centre offset estimated from photos, NOT a hand-eye calibration. -->
-    <!-- Nominal flange radius 40 mm + half camera height 17.5 mm. The camera
-         is physically on flange -Y; +Y was the earlier photo-based guess. -->
-    <xacro:arg name="camera_mount_xyz" default="0 -0.0575 0.015"/>
+    <!-- Camera housing: 90 x 45 x 60 mm measured by user (X length,
+         Y radial height, Z depth along the shooting/tool direction).
+         Centre offset is approximate geometry, NOT a hand-eye calibration. -->
+    <!-- Keep the housing tangent to the nominal 40 mm flange radius on -Y:
+         centre Y = -(40 + 45/2) mm. Keep its rear face at flange Z +5 mm,
+         so the added depth projects forward along +Z. -->
+    <xacro:arg name="camera_mount_xyz" default="0 -0.0625 0.035"/>
     <xacro:arg name="camera_mount_rpy" default="0 0 0"/>
-    <xacro:arg name="camera_size_x" default="0.100"/>
-    <xacro:arg name="camera_size_y" default="0.035"/>
-    <xacro:arg name="camera_size_z" default="0.020"/>
+    <xacro:arg name="camera_size_x" default="0.090"/>
+    <xacro:arg name="camera_size_y" default="0.045"/>
+    <xacro:arg name="camera_size_z" default="0.060"/>
     <xacro:arg name="camera_collision_padding" default="0.003"/>
     <xacro:include filename="$(find fairino_description)/urdf/gemini_pro_placeholder.xacro"/>

File: src/fairino_description/urdf/ydi_j22_placeholder.xacro (robot description, xacro)
@@ -11,5 +11,6 @@
   <xacro:macro name="ydi_j22_placeholder"
                params="parent mount_xyz mount_rpy spacer tcp_xyz tcp_rpy
-                       body_x body_y body_z finger_x finger_y finger_z
+                       body_x body_y body_z body_positive_y_collision_extension
+                       finger_x finger_y finger_z
                        finger_center_x finger_center_y finger_center_z
                        finger_open_multiplier">
@@ -41,6 +42,8 @@
       </visual>
       <collision>
-        <origin xyz="0 0 ${body_z/2}"/>
-        <geometry><box size="${body_x} ${body_y} ${body_z}"/></geometry>
+        <!-- The camera is on flange -Y. Extend only the opposite (+Y) face;
+             shifting by half the extension keeps the camera-side face fixed. -->
+        <origin xyz="0 ${body_positive_y_collision_extension/2} ${body_z/2}"/>
+        <geometry><box size="${body_x} ${body_y + body_positive_y_collision_extension} ${body_z}"/></geometry>
       </collision>
     </link>

Commit message: 修复夹爪问题，完成p4

File: src/fairino3mt_v6_moveit2_config/config/fairino3mt_v6_robot.urdf.xacro (robot description, xacro)
@@ -44,10 +44,11 @@
     <xacro:property name="gripper_finger_z"
       value="${gripper_tcp_flange_xyz[2] - gripper_spacer_m - gripper_finger_proximal_body_z}"/>
-    <xacro:arg name="gripper_finger_center_x" default="0.0205"/>
+    <!-- Centre offset is half the 12 mm finger thickness; with a 0.5 mimic
+         multiplier, the command value equals the clear fingertip aperture. -->
+    <xacro:arg name="gripper_finger_center_x" default="0.006"/>
     <xacro:arg name="gripper_finger_center_y" default="0.021"/>
     <xacro:property name="gripper_finger_center_z"
       value="${gripper_finger_proximal_body_z + gripper_finger_z / 2.0}"/>
-    <!-- (166 mm max span - 53 mm nominal grasp span) / (2 * 130 mm command). -->
-    <xacro:arg name="gripper_finger_open_multiplier" default="0.434615"/>
+    <xacro:arg name="gripper_finger_open_multiplier" default="0.5"/>
     <xacro:include filename="$(find fairino_description)/urdf/ydi_j22_placeholder.xacro"/>
       <xacro:ydi_j22_placeholder parent="flange_link"

File: src/fairino_description/urdf/ydi_j22_placeholder.xacro (robot description, xacro)
@@ -7,6 +7,7 @@
        real collision-free space and contact permission can be limited to the
        fingers. The finger motion is a planning approximation: all four
-       fingers move symmetrically in X from a nominal 29 mm closed opening to
-       the drawing's 166 mm maximum span. -->
+       fingers move symmetrically in X and the command value equals the clear
+       fingertip aperture. The active range is restricted to the 26 mm grasp
+       and 60 mm release states. -->
   <xacro:macro name="ydi_j22_placeholder"
                params="parent mount_xyz mount_rpy spacer tcp_xyz tcp_rpy
@@ -58,5 +59,5 @@
       <origin xyz="0 0 0" rpy="0 0 0"/>
       <axis xyz="1 0 0"/>
-      <limit lower="0.0" upper="0.130" effort="1.0" velocity="0.130"/>
+      <limit lower="0.026" upper="0.060" effort="1.0" velocity="0.060"/>
     </joint>
     <!-- Four independently named contact links. Mimic joints make the two X
