Commit message: 优化细节，加入分类区第二空间，未进行测试验证

File: src/fairino_description/urdf/ydi_j22_placeholder.xacro (robot description, xacro)
@@ -8,5 +8,5 @@
        fingers. The finger motion is a planning approximation: all four
        fingers move symmetrically in X and the command value equals the clear
-       fingertip aperture. The active range is restricted to the 26 mm grasp
+       fingertip aperture. The active range is restricted to the 27 mm grasp
        and 60 mm release states. -->
   <xacro:macro name="ydi_j22_placeholder"
@@ -59,5 +59,5 @@
       <origin xyz="0 0 0" rpy="0 0 0"/>
       <axis xyz="1 0 0"/>
-      <limit lower="0.026" upper="0.060" effort="1.0" velocity="0.060"/>
+      <limit lower="0.027" upper="0.060" effort="1.0" velocity="0.060"/>
     </joint>
     <!-- Four independently named contact links. Mimic joints make the two X
